Commit message: update

File: lite6_description/urdf/lite6.urdf (robot description, URDF)
Before this commit: robot lite6, 11 links, 10 joints
Links:
- removed link link_tcp
- removed link uflite_gripper_link
- link link1: mass 1.169 -> 1.411; geometry collision mesh filename=package://xarm_description/meshes/lite6/collision/link1.stl; visual mesh filename=package://xarm_description/meshes/lite6/visual/link1.stl
- link link2: mass 1.192 -> 1.34; geometry collision mesh filename=package://xarm_description/meshes/lite6/collision/link2.stl; visual mesh filename=package://xarm_description/meshes/lite6/visual/link2.stl
- link link3: mass 0.930 -> 0.953; geometry collision mesh filename=package://xarm_description/meshes/lite6/collision/link3.stl; visual mesh filename=package://xarm_description/meshes/lite6/visual/link3.stl
- link link4: mass 1.31 -> 1.284; geometry collision mesh filename=package://xarm_description/meshes/lite6/collision/link4.stl; visual mesh filename=package://xarm_description/meshes/lite6/visual/link4.stl
- link link5: mass 0.784 -> 0.804; geometry collision mesh filename=package://xarm_description/meshes/lite6/collision/link5.stl; visual mesh filename=package://xarm_description/meshes/lite6/visual/link5.stl
- link link6: mass 0.180 -> 0.13; geometry collision mesh filename=package://xarm_description/meshes/lite6/collision/link6.stl; visual mesh filename=package://xarm_description/meshes/lite6/visual/link6.stl
- link link_base: geometry collision mesh filename=package://xarm_description/meshes/lite6/collision/link_base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; visual mesh filename=package://xarm_description/meshes/lite6/visual/link_base.stl
Joints:
- removed joint gripper_fix
- removed joint joint_tcp
- joint joint1: limit lower=-3.141592653589793 upper=3.141592653589793 effort=50.0 velocity=3.14 -> lower=-6.283185307179586 upper=6.283185307179586 effort=50.0 velocity=3.14
- joint joint4: limit lower=-3.141592653589793 upper=3.141592653589793 effort=32.0 velocity=3.14 -> lower=-6.283185307179586 upper=6.283185307179586 effort=32.0 velocity=3.14
- joint joint6: limit lower=-3.141592653589793 upper=3.141592653589793 effort=20.0 velocity=3.14 -> lower=-6.283185307179586 upper=6.283185307179586 effort=20.0 velocity=3.14

Commit message: made changes to the urdf

File: lite6_description/urdf/lite6.urdf (robot description, URDF)
Before this commit: robot UF_ROBOT, 9 links, 8 joints
Links:
- link link1: geometry collision mesh filename=../meshes/lite6/collision/link1.stl; visual mesh filename=../meshes/lite6/visual/link1.stl
- link link2: geometry collision mesh filename=../meshes/lite6/collision/link2.stl; visual mesh filename=../meshes/lite6/visual/link2.stl
- link link3: geometry collision mesh filename=../meshes/lite6/collision/link3.stl; visual mesh filename=../meshes/lite6/visual/link3.stl
- link link4: geometry collision mesh filename=../meshes/lite6/collision/link4.stl; visual mesh filename=../meshes/lite6/visual/link4.stl
- link link5: geometry collision mesh filename=../meshes/lite6/collision/link5.stl; visual mesh filename=../meshes/lite6/visual/link5.stl
- link link6: geometry collision mesh filename=../meshes/lite6/collision/link6.stl; visual mesh filename=../meshes/lite6/visual/link6.stl
- link link_base: geometry collision mesh filename=../meshes/lite6/collision/link_base.stl; visual mesh filename=../meshes/lite6/visual/base.stl
