Commit message: changed the irdf again to correct the references

File: lite6_description/lite6.urdf (robot description, URDF)
Before this commit: robot UF_ROBOT, 9 links, 8 joints
Links:
- link link1: geometry collision mesh filename=meshes/lite6/collision/link1.stl; visual mesh filename=meshes/lite6/visual/link1.stl
- link link2: geometry collision mesh filename=meshes/lite6/collision/link2.stl; visual mesh filename=meshes/lite6/visual/link2.stl
- link link3: geometry collision mesh filename=../meshes/lite6/collision/link3.stl; visual mesh filename=meshes/lite6/visual/link3.stl
- link link4: geometry collision mesh filename=meshes/lite6/collision/link4.stl; visual mesh filename=meshes/lite6/visual/link4.stl
- link link5: geometry collision mesh filename=meshes/lite6/collision/link5.stl; visual mesh filename=meshes/lite6/visual/link5.stl
- link link6: geometry collision mesh filename=meshes/lite6/collision/link6.stl; visual mesh filename=meshes/lite6/visual/link6.stl
- link link_base: geometry collision mesh filename=meshes/lite6/collision/base.stl; visual mesh filename=meshes/lite6/visual/base.stl

Commit message: changed the irdf again to correct the references

File: lite6_description/lite6.urdf (robot description, URDF)
Before this commit: robot UF_ROBOT, 9 links, 8 joints
Links:
- link link3: geometry collision mesh filename=meshes/lite6/collision/link3.stl; visual mesh filename=meshes/lite6/visual/link3.stl

Commit message: change urdf second

File: lite6_description/lite6.urdf (robot description, URDF)
Before this commit: robot UF_ROBOT, 9 links, 8 joints
Links:
- added link link_gripper; collision mesh filename=meshes/gripper/collision/gripper.stl; visual mesh filename=meshes/gripper/visual/gripper.stl
Joints:
- added joint joint_gripper: type fixed, parent link6, child link_gripper, origin xyz=0 0 0 rpy=0 0 0

Commit message: changed teh urdf again

File: lite6_description/lite6.urdf (robot description, URDF)
Before this commit: robot UF_ROBOT, 10 links, 9 joints
Links:
- link link_gripper: geometry collision mesh filename=meshes/lite6/collision/gripper_lite.stl; visual mesh filename=meshes/lite6/visual/gripper_lite.stl

Commit message: final addition

File: lite6_description/lite6.urdf (robot description, URDF)
Before this commit: robot UF_ROBOT, 10 links, 9 joints
Links:
- removed link link_gripper
- added link base_link, mass 0.1; collision mesh filename=meshes/gripper/base_link.STL; visual mesh filename=meshes/gripper/base_link.STL
- added link left_finger, mass 0.02; collision mesh filename=meshes/gripper/left_finger.STL; visual mesh filename=meshes/gripper/left_finger.STL
- added link left_inner_knuckle, mass 0.03; collision mesh filename=meshes/gripper/left_inner_knuckle.STL; visual mesh filename=meshes/gripper/left_inner_knuckle.STL
- added link left_outer_knuckle, mass 0.05; collision mesh filename=meshes/gripper/left_outer_knuckle.STL; visual mesh filename=meshes/gripper/left_outer_knuckle.STL
- added link right_finger, mass 0.02; collision mesh filename=meshes/gripper/right_finger.STL; visual mesh filename=meshes/gripper/right_finger.STL
- added link right_inner_knuckle, mass 0.03; collision mesh filename=meshes/gripper/right_inner_knuckle.STL; visual mesh filename=meshes/gripper/right_inner_knuckle.STL
- added link right_outer_knuckle, mass 0.05; collision mesh filename=meshes/gripper/right_outer_knuckle.STL; visual mesh filename=meshes/gripper/right_outer_knuckle.STL
Joints:
- added joint left_finger_joint: type revolute, parent base_link, child left_outer_knuckle, origin xyz=0.04 0 0.06 rpy=0 0 0, axis 0 0 1, limit lower=0 upper=0.8 effort=20.0 velocity=2.0
- added joint left_finger_tip_joint: type revolute, parent left_outer_knuckle, child left_finger, origin xyz=0.05 0 0.04 rpy=0 0 0, axis 0 0 1, limit lower=-0.8 upper=0 effort=20.0 velocity=2.0, mimic joint=left_finger_joint multiplier=-1 offset=0
- added joint left_inner_knuckle_joint: type revolute, parent base_link, child left_inner_knuckle, origin xyz=0.04 0 0.06 rpy=0 0 0, axis 0 0 1, limit lower=0 upper=0.8 effort=20.0 velocity=2.0, mimic joint=left_finger_joint multiplier=1 offset=0
- added joint right_finger_joint: type revolute, parent base_link, child right_outer_knuckle, origin xyz=-0.04 0 0.06 rpy=0 0 0, axis 0 0 -1, limit lower=0 upper=0.8 effort=20.0 velocity=2.0, mimic joint=left_finger_joint multiplier=1 offset=0
- added joint right_finger_tip_joint: type revolute, parent right_outer_knuckle, child right_finger, origin xyz=-0.05 0 0.04 rpy=0 0 0, axis 0 0 -1, limit lower=-0.8 upper=0 effort=20.0 velocity=2.0, mimic joint=left_finger_joint multiplier=-1 offset=0
- added joint right_inner_knuckle_joint: type revolute, parent base_link, child right_inner_knuckle, origin xyz=-0.04 0 0.06 rpy=0 0 0, axis 0 0 -1, limit lower=0 upper=0.8 effort=20.0 velocity=2.0, mimic joint=left_finger_joint multiplier=1 offset=0
- joint joint_gripper: child link_gripper -> link_eef

Commit message: made the cahnges

File: lite6_description/lite6.urdf (robot description, URDF)
Before this commit: robot UF_ROBOT, 16 links, 15 joints
Joints:
- joint joint_gripper: child link_eef -> base_link

Commit message: made change

File: lite6_description/lite6.urdf (robot description, URDF)
Before this commit: robot UF_ROBOT, 16 links, 15 joints
Joints:
- joint right_finger_joint: axis 0 0 -1 -> 0 0 1; origin xyz=-0.04 0 0.06 rpy=0 0 0 -> xyz=-0.04 0 0.06 rpy=0 0 3.14159265

Commit message: urdf update rollout

File: lite6_description/lite6.urdf (robot description, URDF)
Before this commit: robot UF_ROBOT, 16 links, 15 joints
Links:
- removed link base_link
- added link link_tcp
- added link xarm_gripper_base_link, mass 0.54156; collision mesh filename=package://xarm_gripper/meshes/base_link_collision.stl; visual mesh filename=package://xarm_gripper/meshes/base_link.stl
- link left_finger: mass 0.02 -> 0.048304; geometry collision mesh filename=package://xarm_gripper/meshes/left_finger.stl; visual mesh filename=package://xarm_gripper/meshes/left_finger.stl
- link left_inner_knuckle: mass 0.03 -> 0.0230125781256706; geometry collision mesh filename=package://xarm_gripper/meshes/left_inner_knuckle.stl; visual mesh filename=package://xarm_gripper/meshes/left_inner_knuckle.stl
- link left_outer_knuckle: mass 0.05 -> 0.033618; geometry collision mesh filename=package://xarm_gripper/meshes/left_outer_knuckle.stl; visual mesh filename=package://xarm_gripper/meshes/left_outer_knuckle.stl
- link right_finger: mass 0.02 -> 0.048304; geometry collision mesh filename=package://xarm_gripper/meshes/right_finger.stl; visual mesh filename=package://xarm_gripper/meshes/right_finger.stl
- link right_inner_knuckle: mass 0.03 -> 0.023013; geometry collision mesh filename=package://xarm_gripper/meshes/right_inner_knuckle.stl; visual mesh filename=package://xarm_gripper/meshes/right_inner_knuckle.stl
- link right_outer_knuckle: mass 0.05 -> 0.033618; geometry collision mesh filename=package://xarm_gripper/meshes/right_outer_knuckle.stl; visual mesh filename=package://xarm_gripper/meshes/right_outer_knuckle.stl
Joints:
- removed joint joint_gripper
- removed joint left_finger_tip_joint
- removed joint right_finger_tip_joint
- added joint drive_joint: type revolute, parent xarm_gripper_base_link, child left_outer_knuckle, origin xyz=0 0.035 0.059098 rpy=0 0 0, axis 1 0 0, limit lower=0 upper=0.85 effort=50 velocity=2
- added joint gripper_fix: type fixed, parent link6, child xarm_gripper_base_link, origin xyz=0 0 0 rpy=0 0 0
- added joint joint_tcp: type fixed, parent xarm_gripper_base_link, child link_tcp, origin xyz=0 0 0.172 rpy=0 0 0
- added joint right_outer_knuckle_joint: type revolute, parent xarm_gripper_base_link, child right_outer_knuckle, origin xyz=0 -0.035 0.059098 rpy=0 0 0, axis -1 0 0, limit lower=0 upper=0.85 effort=50 velocity=2, mimic joint=drive_joint multiplier=1 offset=0
- joint left_finger_joint: axis 0 0 1 -> -1 0 0; child left_outer_knuckle -> left_finger; limit lower=0 upper=0.8 effort=20.0 velocity=2.0 -> lower=0 upper=0.85 effort=50 velocity=2; mimic (none) -> joint=drive_joint multiplier=1 offset=0; origin xyz=0.04 0 0.06 rpy=0 0 0 -> xyz=0 0.035465 0.042039 rpy=0 0 0; parent base_link -> left_outer_knuckle
- joint left_inner_knuckle_joint: axis 0 0 1 -> 1 0 0; limit lower=0 upper=0.8 effort=20.0 velocity=2.0 -> lower=0 upper=0.85 effort=50 velocity=2; mimic joint=left_finger_joint multiplier=1 offset=0 -> joint=drive_joint multiplier=1 offset=0; origin xyz=0.04 0 0.06 rpy=0 0 0 -> xyz=0 0.02 0.074098 rpy=0 0 0; parent base_link -> xarm_gripper_base_link
- joint right_finger_joint: axis 0 0 1 -> 1 0 0; child right_outer_knuckle -> right_finger; limit lower=0 upper=0.8 effort=20.0 velocity=2.0 -> lower=0 upper=0.85 effort=50 velocity=2; mimic joint=left_finger_joint multiplier=1 offset=0 -> joint=drive_joint multiplier=1 offset=0; origin xyz=-0.04 0 0.06 rpy=0 0 3.14159265 -> xyz=0 -0.035465 0.042039 rpy=0 0 0; parent base_link -> right_outer_knuckle
- joint right_inner_knuckle_joint: axis 0 0 -1 -> -1 0 0; limit lower=0 upper=0.8 effort=20.0 velocity=2.0 -> lower=0 upper=0.85 effort=50 velocity=2; mimic joint=left_finger_joint multiplier=1 offset=0 -> joint=drive_joint multiplier=1 offset=0; origin xyz=-0.04 0 0.06 rpy=0 0 0 -> xyz=0 -0.02 0.074098 rpy=0 0 0; parent base_link -> xarm_gripper_base_link

Commit message: CHANGE DONE

File: lite6_description/lite6.urdf (robot description, URDF)
Before this commit: robot UF_ROBOT, 17 links, 16 joints
Links:
- link left_finger: geometry collision mesh filename=meshes/gripper/left_finger.STL; visual mesh filename=meshes/gripper/left_finger.STL
- link left_inner_knuckle: geometry collision mesh filename=meshes/gripper/left_inner_knuckle.STL; visual mesh filename=meshes/gripper/left_inner_knuckle.STL
- link left_outer_knuckle: geometry collision mesh filename=meshes/gripper/left_outer_knuckle.STL; visual mesh filename=meshes/gripper/left_outer_knuckle.STL
- link right_finger: geometry collision mesh filename=meshes/gripper/right_finger.STL; visual mesh filename=meshes/gripper/right_finger.STL
- link right_inner_knuckle: geometry collision mesh filename=meshes/gripper/right_inner_knuckle.STL; visual mesh filename=meshes/gripper/right_inner_knuckle.STL
- link right_outer_knuckle: geometry collision mesh filename=meshes/gripper/right_outer_knuckle.stl; visual mesh filename=meshes/gripper/right_outer_knuckle.stl
- link xarm_gripper_base_link: geometry collision mesh filename=meshes/gripper/base_link_collision.STL; visual mesh filename=meshes/gripper/base_link.STL

Commit message: dfdfd

File: lite6_description/lite6.urdf (robot description, URDF)
Before this commit: robot UF_ROBOT, 17 links, 16 joints
Links:
- link xarm_gripper_base_link: geometry collision mesh filename=meshes/gripper/base_link.STL; visual mesh filename=meshes/gripper/base_link.STL

Commit message: sasasa

File: lite6_description/lite6.urdf (robot description, URDF)
Before this commit: robot UF_ROBOT, 17 links, 16 joints
Links:
- link right_outer_knuckle: geometry collision mesh filename=meshes/gripper/right_outer_knuckle.STL; visual mesh filename=meshes/gripper/right_outer_knuckle.STL

Commit message: change

File: lite6_description/lite6.urdf (robot description, URDF)
Before this commit: robot UF_ROBOT, 11 links, 11 joints
Joints:
- removed joint drive_joint
